File: KiCAD Files/MOSFET&SENSOR.kicad_sch (KiCad schematic)
At the start: 36 parts, among them Q1 IRLZ44N, Q2 IRLZ44N, Q3 IRLZ44N, Q4 IRLZ44N, U4 ACS712xLCTR-05B, U5 ACS712xLCTR-05B, U6 ACS712xLCTR-05B, U7 ACS712xLCTR-05B

Commit message: update
Parts:
- removed C10, C13, C14, C9: 100n, Capacitor_SMD:C_0603_1608Metric, symbol Device:C
- removed C11, C12, C15, C16: 1n, Capacitor_SMD:C_0603_1608Metric, symbol Device:C
- removed U4, U5, U6, U7: ACS712xLCTR-05B, Package_SO:SOIC-8_3.9x4.9mm_P1.27mm, symbol Sensor_Current:ACS712xLCTR-05B
Connections:
- net at F3.1: now also R17.1
- net at R11.1: now also F1.1
- net at R12.1: now also F2.1
- net at R18.1: now also F4.1
Other:
- moved on the sheet: BT1, BT2, BT3, BT4, F1, F2, F3, F4, Q1, Q2, Q3, Q4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
