File: KiCAD Files/BatteryDischargerV1.kicad_pcb (KiCad board)
At the start: 2 copper layers, 100 x 160 mm, 55 parts, among them J1 USBasp, J2 OLED, J3 UART, Q1 IRLZ44N, Q2 IRLZ44N, Q3 IRLZ44N, Q4 IRLZ44N, SW1 SW_Push, SW2 SW_Push, U1 ATmega328-A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

Commit message: update
Routing:
- net +3V3: track 30.4 -> 29.3 mm
Other:
- board text added: "JLCJLCJLCJLC"
Changed lines of the file:
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@@
   (gr_arc (start 56.25 22.75) (mid 57.421573 19.921573) (end 60.25 18.75) (layer "Edge.Cuts") (width 0.1))
   (gr_arc (start 152.25 18.75) (mid 155.078427 19.921573) (end 156.25 22.75) (layer "Edge.Cuts") (width 0.1))
+  (gr_text "JLCJLCJLCJLC" (at 94.8 68 90) (layer "F.SilkS")
+    (effects (font (size 1.5 1.5) (thickness 0.2)))
+  )
   (segment (start 90.6444 160.25) (end 87.8944 163) (width 0.3556) (layer "F.Cu") (net 1))
   (segment (start 99.25 159.75) (end 98.75 160.25) (width 0.3556) (layer "F.Cu") (net 1))
@@
   (segment (start 106.65 168.4) (end 106.25 168) (width 0.3556) (layer "F.Cu") (net 7))
   (segment (start 106.65 167.35) (end 106.65 167.6) (width 0.3556) (layer "F.Cu") (net 7))
-  (segment (start 101.5 137.25) (end 84 137.25) (width 0.762) (layer "F.Cu") (net 8))
-  (segment (start 105.04 140.79) (end 101.5 137.25) (width 0.762) (layer "F.Cu") (net 8))
-  (segment (start 83.225 138.025) (end 83.225 140.25) (width 0.762) (layer "F.Cu") (net 8))
-  (segment (start 84 137.25) (end 83.225 138.025) (width 0.762) (layer "F.Cu") (net 8))
-  (segment (start 105.04 145.4095) (end 105.04 140.79) (width 0.762) (layer "F.Cu") (net 8))
-  (segment (start 123.25 109.77) (end 123.25 98.002) (width 0.762) (layer "F.Cu") (net 9))
-  (segment (start 123.25 98.002) (end 124.55 96.702) (width 0.762) (layer "F.Cu") (net 9))
-  (segment (start 100.25 98.002) (end 101.55 96.702) (width 0.762) (layer "F.Cu") (net 10))
-  (segment (start 100.25 109.77) (end 100.25 98.002) (width 0.762) (layer "F.Cu") (net 10))
+  (segment (start 105.04 142.71) (end 105.04 145.4095) (width 0.762) (layer "F.Cu") (net 8))
+  (segment (start 83.225 140.25) (end 83.225 138.025) (width 0.762) (layer "F.Cu") (net 8))
+  (segment (start 83.225 138.025) (end 84 137.25) (width 0.762) (layer "F.Cu") (net 8))
+  (segment (start 99.58 137.25) (end 105.04 142.71) (width 0.762) (layer "F.Cu") (net 8))
+  (segment (start 84 137.25) (end 99.58 137.25) (width 0.762) (layer "F.Cu") (net 8))
+  (segment (start 123.25 109.77) (end 123.25 98.002) (width 1.2) (layer "F.Cu") (net 9))
+  (segment (start 123.25 98.002) (end 124.55 96.702) (width 1.2) (layer "F.Cu") (net 9))
+  (segment (start 100.25 98.002) (end 101.55 96.702) (width 1.2) (layer "F.Cu") (net 10))
+  (segment (start 100.25 109.77) (end 100.25 98.002) (width 1.2) (layer "F.Cu") (net 10))
   (segment (start 147.9975 143.2475) (end 147.9975 144.92) (width 0.3556) (layer "F.Cu") (net 11))
   (segment (start 104.25 150.75) (end 105.25 149.75) (width 0.3556) (layer "F.Cu") (net 11))
@@
   (segment (start 78.25 131.675) (end 78.25 130.75) (width 0.3556) (layer "F.Cu") (net 20))
   (segment (start 79.79 109.75) (end 81.25 109.75) (width 0.3556) (layer "F.Cu") (net 20))
-  (segment (start 77.25 98.002) (end 78.55 96.702) (width 0.762) (layer "F.Cu") (net 21))
-  (segment (start 77.25 109.75) (end 77.25 98.002) (width 0.762) (layer "F.Cu") (net 21))
+  (segment (start 77.25 98.002) (end 78.55 96.702) (width 1.2) (layer "F.Cu") (net 21))
+  (segment (start 77.25 109.75) (end 77.25 98.002) (width 1.2) (layer "F.Cu") (net 21))
   (segment (start 129 129.52) (end 128.25 130.27) (width 0.3556) (layer "F.Cu") (net 22))
   (segment (start 122.25 130.77) (end 122.75 130.27) (width 0.3556) (layer "F.Cu") (net 22))
@@
   (segment (start 148.79 109.77) (end 150.25 109.77) (width 0.3556) (layer "F.Cu") (net 25))
   (segment (start 145.75 130.27) (end 146.75 130.27) (width 0.3556) (layer "F.Cu") (net 25))
-  (segment (start 146.25 109.77) (end 146.25 98.002) (width 0.762) (layer "F.Cu") (net 26))
-  (segment (start 146.25 98.002) (end 147.55 96.702) (width 0.762) (layer "F.Cu") (net 26))
+  (segment (start 146.25 109.77) (end 146.25 98.002) (width 1.2) (layer "F.Cu") (net 26))
+  (segment (start 146.25 98.002) (end 147.55 96.702) (width 1.2) (layer "F.Cu") (net 26))
   (segment (start 129.75 167) (end 142.25 167) (width 1.2) (layer "F.Cu") (net 27))
   (segment (start 85.425 167) (end 83 167) (width 0.4572) (layer "F.Cu") (net 28))
