File: KiCAD Files/BatteryDischargerV1.kicad_pcb (KiCad board)
At the start: 2 copper layers, 98 x 98 mm, 74 parts, among them J1 USBasp, J2 ST7789, J3 UART, Q1 IRLZ44N, Q2 IRLZ44N, Q3 IRLZ44N, Q4 IRLZ44N, SW1 SW_Push, SW2 SW_Push, SW3 SW_Push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

Commit message: update
Parts:
- removed C4: 100n, Capacitor_SMD:C_0805_2012Metric
- removed R6: 100, Resistor_SMD:R_0603_1608Metric
- removed SW3: SW_Push, Button_Switch_SMD:SW_SPST_TL3342
- H1, Q1, Q2, Q3, Q4, R11, R12, R17, R18: moved to B.Cu
- moved F3 256.1 mm to (88.8, 122.2), turned to 180 degrees
- moved F2 253.2 mm to (111.8, 122.2), turned to 180 degrees
- moved U6 251.5 mm to (98.8, 134.0)
- moved F4 251.0 mm to (134.8, 122.5), turned to 180 degrees
- moved F1 238.7 mm to (65.8, 122.2), turned to 180 degrees
- moved J2 236.0 mm to (106.2, 139.7)
- moved J3 233.5 mm to (145.4, 163.0)
- moved SW2 228.6 mm to (71.5, 165.5)
- moved SW1 224.0 mm to (126.8, 167.0)
- moved R13 223.9 mm to (77.2, 120.2), turned to 180 degrees
- moved R15 222.0 mm to (77.2, 118.0)
- moved C16 218.3 mm to (150.0, 135.2), turned to -90 degrees
- moved R19 208.2 mm to (100.2, 120.2), turned to 180 degrees
- moved Q2 207.0 mm to (120.7, 109.8)
- moved Q4 206.9 mm to (143.7, 109.8)
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Connections:
- C5 pad 1: VBAT2 -> VBAT1
- L2 pad 1: VBAT2 -> VBAT1
- U3 pad 4: VBAT2 -> VBAT1
- U3 pad 5: VBAT2 -> VBAT1
Routing:
- net Net-(R18-Pad1): track 0.00 -> 108.1 mm
- net Net-(R17-Pad1): track 0.00 -> 108.1 mm
- net Net-(R12-Pad1): track 0.00 -> 108.1 mm
- net Net-(R11-Pad1): track 0.00 -> 108.1 mm
- net MOSFET2: track 0.00 -> 45.2 mm
- net MOSFET1: track 0.00 -> 38.3 mm
- net Net-(Q4-Pad1): track 0.00 -> 14.5 mm
- net Net-(Q3-Pad1): track 0.00 -> 14.3 mm
- net Net-(Q2-Pad1): track 0.00 -> 14.3 mm
- net Net-(Q1-Pad1): track 0.00 -> 14.0 mm
- net Net-(Q4-Pad2): track 0.00 -> 13.6 mm
- net Net-(Q3-Pad2): track 0.00 -> 13.6 mm
- net Net-(Q2-Pad2): track 0.00 -> 13.6 mm
- net Net-(Q1-Pad2): track 0.00 -> 13.6 mm
- net PB5: track 0.00 -> 11.6 mm
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- added copper zone on B.Cu, net GND
Other:
- board size 98 x 98 mm -> 100 x 160 mm

Commit message: update
Parts:
- removed C10, C13, C14, C9: 100n, Capacitor_SMD:C_0603_1608Metric
- removed C11, C12, C15, C16: 1n, Capacitor_SMD:C_0603_1608Metric
- removed R1, R2, R3, R5: 220, Resistor_SMD:R_0603_1608Metric
- removed U4, U5, U6, U7: ACS712xLCTR-05B, Package_SO:SOIC-8_3.9x4.9mm_P1.27mm
- C1, C2, C3, CD1, CD2: footprint Capacitor_SMD:C_0805_2012Metric -> Capacitor_SMD:C_0603_1608Metric
- J2: value ST7789 -> OLED; footprint Footprint:ST7789 -> Footprint:OLED
- Q1, Q2, Q3, Q4: moved to F.Cu
- moved C8 28.0 mm to (81.8, 140.2), turned to 180 degrees
- moved C7 18.9 mm to (81.8, 156.0)
- moved U2 18.0 mm to (81.8, 148.0)
- moved CD2 17.3 mm to (86.2, 172.0), turned to 180 degrees
- moved R15 14.5 mm to (76.2, 132.5), turned to -90 degrees
- moved R16 14.5 mm to (122.2, 132.5), turned to -90 degrees
- moved R21 14.5 mm to (99.2, 132.5), turned to -90 degrees
- moved R22 14.5 mm to (145.2, 132.5), turned to -90 degrees
- moved C6 12.5 mm to (64.2, 157.0)
- moved R13 12.3 mm to (78.2, 132.5), turned to 90 degrees
- moved R14 12.3 mm to (124.2, 132.5), turned to 90 degrees
- moved R19 12.3 mm to (101.2, 132.5), turned to 90 degrees
- moved R20 12.3 mm to (147.2, 132.5), turned to 90 degrees
- moved CD1 12.1 mm to (126.5, 170.0)
- moved L2 12.0 mm to (64.0, 150.5)
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Connections:
- net INT0 renamed PD2/INT0
- net INT1 renamed PD3/INT1
- net MOSI renamed PB3
- C3 pad 1: +5V -> /AREF
- F3 pad 1: Net-(F3-Pad1) -> Net-(R17-Pad1)
- J2 pad 3: Net-(J2-Pad3) -> SCL
- J2 pad 4: Net-(J2-Pad4) -> SDA
- J3 pad 1: /TX -> GND
- J3 pad 3: GND -> /TX
- LS1 pad 1: Net-(LS1-Pad1) -> /BUZZER
- R11 pad 1: Net-(R11-Pad1) -> Net-(F1-Pad1)
- R12 pad 1: Net-(R12-Pad1) -> Net-(F2-Pad1)
- R18 pad 1: Net-(R18-Pad1) -> Net-(F4-Pad1)
- U1 pad 10: MOSFET3 -> MOSFET4
- U1 pad 11: MOSFET4 -> MOSFET3
- U1 pad 12: PB0 -> unconnected-(U1-Pad12)
- U1 pad 13: PB1 -> unconnected-(U1-Pad13)
- U1 pad 14: Net-(LS1-Pad1) -> MOSFET2
- U1 pad 19: IBAT3 -> unconnected-(U1-Pad19)
- U1 pad 20: +5V -> /AREF
- U1 pad 22: IBAT4 -> unconnected-(U1-Pad22)
- U1 pad 27: IBAT1 -> SDA
- U1 pad 28: IBAT2 -> SCL
- U1 pad 9: MOSFET2 -> /BUZZER
Routing:
- net Net-(R18-Pad1): track 108.1 -> 0.00 mm
- net Net-(R12-Pad1): track 108.1 -> 0.00 mm
- net Net-(R11-Pad1): track 108.1 -> 0.00 mm
- net Net-(F4-Pad1): track 8.03 -> 107.6 mm
- net Net-(F2-Pad1): track 8.13 -> 107.6 mm
- net Net-(F1-Pad1): track 8.13 -> 107.6 mm
- net RESET: track 0.00 -> 91.9 mm
- net PB5: track 11.6 -> 99.2 mm
- net +5V: track 2.78 -> 75.2 mm
- net PB4: track 10.6 -> 79.8 mm
- net VBAT1: track 11.2 -> 69.8 mm, vias 0 -> 2
- net VBAT2: track 11.2 -> 68.4 mm, vias 0 -> 4
- net PB3: track 0.00 -> 53.6 mm
- net /TX: track 0.00 -> 52.8 mm
- net MOSFET4: track 0.00 -> 50.4 mm, vias 0 -> 2
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- added copper zone on F.Cu, net +3V3
- added copper zone on F.Cu, net +5V
- added copper zone on F.Cu, net /L_OUT
- added copper zone on F.Cu, net GND
- added copper zone on F.Cu, net VBAT1

Commit message: update
Parts:
- moved CD2 2.85 mm to (87.0, 169.2)
- moved R4 2.25 mm to (103.5, 165.8)
- moved CD1 1.12 mm to (125.5, 169.5)
- moved R7 1.00 mm to (125.5, 167.0)
- moved R8 0.75 mm to (87.0, 167.0)
- moved SW1 0.25 mm to (129.5, 167.0)
- moved J2 0.09 mm to (102.5, 145.5)
Connections:
- H1 pad 1: (no net) -> unconnected-(H1-Pad1)
- H2 pad 1: (no net) -> unconnected-(H2-Pad1)
- H3 pad 1: (no net) -> unconnected-(H3-Pad1)
- H4 pad 1: (no net) -> unconnected-(H4-Pad1)
- J3 pad 2: /RX -> /TX
- J3 pad 3: /TX -> /RX
- U1 pad 30: /TX -> /RX
- U1 pad 31: /RX -> /TX
Routing:
- net +5V: track 75.2 -> 188.1 mm, vias 0 -> 3
- net MOSFET1: track 0.00 -> 110.7 mm, vias 0 -> 6
- net VBAT3: track 0.00 -> 83.3 mm, vias 0 -> 4
- net VBAT4: track 0.00 -> 76.3 mm, vias 0 -> 4
- net SDA: track 0.00 -> 33.9 mm, vias 0 -> 1
- net PD2/INT0: track 0.00 -> 23.9 mm
- net PD3/INT1: track 9.52 -> 32.6 mm, vias 0 -> 2
- net SCL: track 0.00 -> 18.5 mm, vias 0 -> 1
- net /RX: track 41.0 -> 56.1 mm
- net MOSFET2: track 31.0 -> 22.6 mm, vias 2 -> 4
- net VBAT2: track 68.4 -> 76.0 mm, vias 4 -> 6
- net GND: track 23.0 -> 30.4 mm, vias 48 -> 52
- net Net-(R7-Pad1): track 12.5 -> 15.7 mm
- net PB4: track 79.8 -> 82.2 mm
- net /TX: track 52.8 -> 54.8 mm
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Other:
- board text added: "GND"
- board text added: "RX"
- board text added: "TX"
