File: KiCAD Files/BatteryDischargerV1.kicad_sch (KiCad schematic)
At the start: 0 parts

Commit message: update
Parts:
- added BT? (x4): 4V2 - 18650, symbol Device:Battery_Cell
- added F? (x4): 2A, symbol Device:Fuse
- added Q? (x4): IRLZ44N, Package_TO_SOT_THT:TO-220-3_Vertical, symbol Transistor_FET:IRLZ44N
- added R? (x4): R100, symbol Device:R_Small
- added R? (x4): 10k, symbol Device:R_Small
- added R? (x4): 3R3, 10W, symbol Device:R
- added U?: ATmega328-A, Package_QFP:TQFP-32_7x7mm_P0.8mm, symbol MCU_Microchip_ATmega:ATmega328-A
Connections:
- new net: F?.1, R?.1 (x4)
- new net: Q?.1 (G), R?.1, R?.2 (x4)
- new net: Q?.2 (D), R?.2 (x4)
- new net: U?.21 (GND), U?.3 (GND), U?.5 (GND)
- new net: U?.4 (VCC), U?.6 (VCC)
- new net GND: BT?.2 (-), BT?.2 (-), BT?.2 (-), BT?.2 (-), Q?.3 (S), Q?.3 (S), Q?.3 (S), Q?.3 (S), R?.2, R?.2, R?.2, R?.2
- new net MOSFET1: R?.1
- new net MOSFET2: R?.1
- new net MOSFET3: R?.1
- new net MOSFET4: R?.1
- new net VBAT1: BT?.1 (+), F?.2
- new net VBAT2: BT?.1 (+), F?.2
- new net VBAT3: BT?.1 (+), F?.2
- new net VBAT4: BT?.1 (+), F?.2

Commit message: Update BatteryDischargerV1.kicad_sch
Parts:
- removed BT? (x3): 4V2 - 18650, symbol Device:Battery_Cell
- removed F? (x3): 2A, symbol Device:Fuse
- removed Q? (x3): IRLZ44N, Package_TO_SOT_THT:TO-220-3_Vertical, symbol Transistor_FET:IRLZ44N
- removed R? (x3): 10k, symbol Device:R_Small
- removed R? (x3): R100, symbol Device:R_Small
- removed R? (x3): 3R3, 10W, symbol Device:R
- removed U?: ATmega328-A, Package_QFP:TQFP-32_7x7mm_P0.8mm, symbol MCU_Microchip_ATmega:ATmega328-A
- added BT? (x3): 4V2 - 18650, symbol Device:Battery_Cell
- added C? (x4): 100n, Capacitor_SMD:C_0805_2012Metric, symbol Device:C_Small
- added C? (x4): 100n, Capacitor_SMD:C_0603_1608Metric, symbol Device:C
- added C? (x4): 1n, Capacitor_SMD:C_0603_1608Metric, symbol Device:C
- added C? (x2): 22u / 16V, Capacitor_SMD:C_1210_3225Metric, symbol Device:C_Small
- added D?: SS12, Diode_SMD:D_SMA, symbol Device:D_Schottky_Small
- added F? (x3): 2A, symbol Device:Fuse
- added J?: UART, symbol Connector_Generic:Conn_01x03
- added J?: USBasp, Connector_PinSocket_1.27mm:PinSocket_2x03_P1.27mm_Vertical, symbol Connector_Generic:Conn_02x03_Odd_Even
- added L?: 4R7, Footprints:Inductor_4mm(5x5mm pads), symbol Device:L_Small
- added L?: 10u, Inductor_SMD:L_1206_3216Metric, symbol Device:L_Small
- added LS?: Buzzer, CNLJS:KLJ-1102, symbol Device:Speaker
- added Q? (x3): IRLZ44N, Package_TO_SOT_THT:TO-220-3_Vertical, symbol Transistor_FET:IRLZ44N
- added R? (x3): 3R3, 10W, symbol Device:R
- added R?: 100k, Resistor_SMD:R_0603_1608Metric, symbol Device:R_Small
- added R? (x3): 10k, symbol Device:R_Small
- added R? (x3): R100, symbol Device:R_Small
- added R?: 10k, Resistor_SMD:R_0603_1608Metric, symbol Device:R_Small
- added R?: 100, Resistor_SMD:R_0603_1608Metric, symbol Device:R_Small
- added R?: 13k3, Resistor_SMD:R_0603_1608Metric, symbol Device:R_Small
- added SW?: SW_Push, Button_Switch_SMD:SW_SPST_TL3342, symbol Switch:SW_Push
- added U? (x4): ACS712xLCTR-05B, Package_SO:SOIC-8_3.9x4.9mm_P1.27mm, symbol Sensor_Current:ACS712xLCTR-05B
- added U?: ATmega328-A, Package_QFP:TQFP-32_7x7mm_P0.8mm, symbol MCU_Microchip_ATmega:ATmega328-A
- added U?: MT3608, Package_TO_SOT_SMD:SOT-23-6, symbol Regulator_Switching:MT3608
- added Y?: 16MHz, CNLJS:CSTCE16M0V53-R0, symbol Device:Resonator_Small
Connections:
- net GND: now also BT?.2 (-), BT?.2 (-), BT?.2 (-), C?.2, C?.2, C?.2, C?.2, C?.2, J?.3 (Pin_3), J?.6 (Pin_6), LS?.2, Q?.3 (S), Q?.3 (S), Q?.3 (S), R?.1, R?.2, R?.2, R?.2, R?.2, SW?.1, U?.2 (GND), U?.21 (GND), U?.3 (GND), U?.5 (GND), Y?.2
- net MOSFET2: now also R?.1
- net MOSFET3: now also R?.1
- net MOSFET4: now also R?.1
- net VBAT1: now also U?.23 (PC0)
- net VBAT2: now also BT?.1 (+), C?.1, F?.2, L?.1, U?.24 (PC1), U?.4 (EN), U?.5 (IN)
- net VBAT3: now also BT?.1 (+), F?.2, U?.25 (PC2)
- net VBAT4: now also BT?.1 (+), F?.2, U?.26 (PC3)
- net at F?.1: now also U?.3 (IP-), U?.4 (IP-); no longer R?.1
- new net: R?.1, U?.1 (IP+), U?.2 (IP+) (x4)
- new net: Q?.2 (D), R?.2 (x3)
- new net: C?.2, R?.2
- new net: Q?.1 (G), R?.1, R?.2 (x3)
- new net: F?.1, U?.3 (IP-), U?.4 (IP-) (x3)
- new net: C?.1, U?.6 (FILTER) (x4)
- new net: U?.8 (XTAL2/PB7), Y?.1
- new net: U?.7 (XTAL1/PB6), Y?.3
- new net: LS?.1, U?.14 (PB2)
- new net: C?.1, L?.2, U?.18 (AVCC)
- new net +5V: C?.1, C?.1, C?.1, C?.1, C?.1, C?.1, C?.1, D?.1 (K), L?.1, R?.1, R?.2, U?.20 (AREF), U?.4 (VCC), U?.6 (VCC), U?.8 (VCC), U?.8 (VCC), U?.8 (VCC), U?.8 (VCC)
- new net FB: R?.1, R?.2, U?.3 (FB)
- new net GNDA: C?.2, C?.2, C?.2, C?.2, C?.2, C?.2, C?.2, C?.2, U?.5 (GND), U?.5 (GND), U?.5 (GND), U?.5 (GND)
- new net IBAT1: U?.27 (PC4), U?.7 (VIOUT)
- new net IBAT2: U?.28 (PC5), U?.7 (VIOUT)
- new net IBAT3: U?.19 (ADC6), U?.7 (VIOUT)
- new net IBAT4: U?.22 (ADC7), U?.7 (VIOUT)
- new net L_OUT: D?.2 (A), L?.2, U?.1 (SW)
- new net MISO: J?.1 (Pin_1), U?.16 (PB4)
- new net MOSI: J?.4 (Pin_4), U?.15 (PB3)
- new net RESET: C?.1, J?.5 (Pin_5), R?.1, SW?.2, U?.29 (~{RESET}/PC6)
- new net RX: J?.2 (Pin_2), U?.31 (PD1)
- new net SCK: J?.3 (Pin_3), U?.17 (PB5)
- new net TX: J?.1 (Pin_1), U?.30 (PD0)
- no-connect marks 0 -> 9
Other:
- note added: "USBasp port"
- moved on the sheet: BT?, F?, Q?, R?

Commit message: update
Parts:
- removed BT? (x4): 4V2 - 18650, symbol Device:Battery_Cell
- removed C? (x4): 100n, Capacitor_SMD:C_0603_1608Metric, symbol Device:C
- removed C? (x4): 1n, Capacitor_SMD:C_0603_1608Metric, symbol Device:C
- removed F? (x4): 2A, symbol Device:Fuse
- removed J?: USBasp, Connector_PinSocket_1.27mm:PinSocket_2x03_P1.27mm_Vertical, symbol Connector_Generic:Conn_02x03_Odd_Even
- removed Q? (x4): IRLZ44N, Package_TO_SOT_THT:TO-220-3_Vertical, symbol Transistor_FET:IRLZ44N
- removed R? (x4): 3R3, 10W, symbol Device:R
- removed R? (x4): R100, symbol Device:R_Small
- removed R? (x4): 10k, symbol Device:R_Small
- removed U? (x4): ACS712xLCTR-05B, Package_SO:SOIC-8_3.9x4.9mm_P1.27mm, symbol Sensor_Current:ACS712xLCTR-05B
- added C7, C8: 10u, Capacitor_SMD:C_1210_3225Metric, symbol Device:C_Small
- added CD1, CD2: 100n, Capacitor_SMD:C_0805_2012Metric, symbol Device:C
- added H1, H2, H3, H4: MountingHole, MountingHole:MountingHole_3.2mm_M3_Pad_Via, symbol Mechanical:MountingHole
- added J1: USBasp, Connector_IDC:IDC-Header_2x05_P2.54mm_Vertical, symbol Connector_Generic:Conn_02x05_Odd_Even
- added J2: ST7789, Footprint:ST7789, symbol Connector_Generic:Conn_01x07
- added R1, R2, R3, R5: 220, Resistor_SMD:R_0603_1608Metric, symbol Device:R_Small
- added R7, R8: 100, Resistor_SMD:R_0603_1608Metric, symbol Device:R
- added SW1, SW2: SW_Push, Footprint:Omron_B3F-12x12mm, symbol Switch:SW_Push
- added U2: AMS1117-3.3, Package_TO_SOT_SMD:SOT-223-3_TabPin2, symbol Regulator_Linear:AMS1117-3.3
- J3: renamed from J?; footprint (none) -> Connector_PinHeader_2.54mm:PinHeader_1x03_P2.54mm_Horizontal
- L2: renamed from L?; footprint Footprints:Inductor_4mm(5x5mm pads) -> Footprint:Inductor_4mm(5x5mm pads)
- LS1: renamed from LS?; footprint CNLJS:KLJ-1102 -> Buzzer_Beeper:Buzzer_TDK_PS1240P02BT_D12.2mm_H6.5mm
- Y1: renamed from Y?; footprint CNLJS:CSTCE16M0V53-R0 -> Footprint:CSTCE16M0V53-R0
- gave numbers to parts that had none: 15
Connections:
- net +5V: now also C7.1, J1.2 (Pin_2), U2.3 (VI)
- net GND: now also C4.2, C7.2, C8.2, CD1.2, CD2.2, J1.10 (Pin_10), J1.3 (Pin_3), J1.4 (Pin_4), J1.6 (Pin_6), J1.8 (Pin_8), J2.1 (Pin_1), SW1.2, SW2.2, U2.1 (GND); no longer SW3.1
- net MOSFET1: now also U1.2 (PD4)
- net MOSFET2: now also U1.9 (PD5)
- net MOSFET3: now also U1.10 (PD6)
- net MOSFET4: now also U1.11 (PD7)
- net MOSI: now also J1.1 (Pin_1)
- net RESET: now also J1.5 (Pin_5)
- net at R6.2: now also SW3.1; no longer C4.2
- net INT1: now reaches U1.1 (PD3)
- net INT1: now also CD2.1, R8.2
- net PB0: now reaches U1.12 (PB0)
- net PB0: now also R3.1
- net PB1: now reaches U1.13 (PB1)
- net PB1: now also R5.1
- net INT0: now reaches U1.32 (PD2)
- net INT0: now also CD1.1, R7.2
- net MISO renamed PB4
- net PB4: now also J1.9 (Pin_9), R2.1
- net SCK renamed PB5
- net PB5: now also J1.7 (Pin_7), R1.1
- new net: J2.5 (Pin_5), R3.2
- new net: R8.1, SW2.1
- new net: J2.6 (Pin_6), R5.2
- new net: J2.4 (Pin_4), R2.2
- new net: R7.1, SW1.1
- new net: J2.3 (Pin_3), R1.2
- new net +3V3: C8.1, J2.2 (Pin_2), U2.2 (VO)
- no-connect marks 9 -> 1
Other:
- added sheet MOSFET&SENSOR (MOSFET&SENSOR.kicad_sch)
- note added: "ST7789"
- note added: "TIPKALA"
- moved on the sheet: C1, C2, C3, C4, J3, L1, LS1, R4, R6, SW3, U1, Y1

Commit message: update
Parts:
- removed C4: 100n, Capacitor_SMD:C_0805_2012Metric, symbol Device:C_Small
- removed R6: 100, Resistor_SMD:R_0603_1608Metric, symbol Device:R_Small
- removed SW3: SW_Push, Button_Switch_SMD:SW_SPST_TL3342, symbol Switch:SW_Push
Connections:
- net VBAT1: now also C5.1, L2.1, U3.4 (EN), U3.5 (IN)
- net VBAT2: no longer C5.1, L2.1, U3.4 (EN), U3.5 (IN)
Changed lines of the file:
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@@
   (junction (at 69.215 157.48) (diameter 0) (color 0 0 0 0)
   )
-  (junction (at 30.48 104.14) (diameter 0) (color 0 0 0 0)
-  )
   (junction (at 42.545 74.295) (diameter 0) (color 0 0 0 0)
   )
@@
   )
   (junction (at 69.215 142.875) (diameter 0) (color 0 0 0 0)
-  )
-  (junction (at 48.895 100.33) (diameter 0) (color 0 0 0 0)
   )
   (junction (at 107.95 33.655) (diameter 0) (color 0 0 0 0)
@@
     (stroke (width 0) (type default) (color 0 0 0 0))
   )
-  (wire (pts (xy 48.895 104.14) (xy 48.895 100.33))
-    (stroke (width 0) (type default) (color 0 0 0 0))
-  )
   (wire (pts (xy 40.005 69.215) (xy 42.545 69.215))
     (stroke (width 0) (type default) (color 0 0 0 0))
@@
     (stroke (width 0) (type default) (color 0 0 0 0))
   )
-  (wire (pts (xy 30.48 104.14) (xy 30.48 106.045))
-    (stroke (width 0) (type default) (color 0 0 0 0))
-  )
   (wire (pts (xy 132.08 149.86) (xy 138.43 149.86))
     (stroke (width 0) (type default) (color 0 0 0 0))
@@
     (stroke (width 0) (type default) (color 0 0 0 0))
   )
-  (wire (pts (xy 30.48 100.33) (xy 31.75 100.33))
-    (stroke (width 0) (type default) (color 0 0 0 0))
-  )
   (wire (pts (xy 110.49 157.48) (xy 110.49 158.75))
     (stroke (width 0) (type default) (color 0 0 0 0))
@@
     (stroke (width 0) (type default) (color 0 0 0 0))
   )
-  (wire (pts (xy 30.48 104.14) (xy 40.005 104.14))
-    (stroke (width 0) (type default) (color 0 0 0 0))
-  )
   (wire (pts (xy 28.575 141.605) (xy 28.575 142.875))
     (stroke (width 0) (type default) (color 0 0 0 0))
@@
     (stroke (width 0) (type default) (color 0 0 0 0))
   )
-  (wire (pts (xy 36.83 100.33) (xy 37.465 100.33))
-    (stroke (width 0) (type default) (color 0 0 0 0))
-  )
   (wire (pts (xy 156.845 94.615) (xy 156.845 92.075))
     (stroke (width 0) (type default) (color 0 0 0 0))
   )
-  (wire (pts (xy 47.625 100.33) (xy 48.895 100.33))
-    (stroke (width 0) (type default) (color 0 0 0 0))
-  )
   (wire (pts (xy 42.545 74.295) (xy 42.545 76.835))
     (stroke (width 0) (type default) (color 0 0 0 0))
@@
     (stroke (width 0) (type default) (color 0 0 0 0))
   )
-  (wire (pts (xy 30.48 100.33) (xy 30.48 104.14))
-    (stroke (width 0) (type default) (color 0 0 0 0))
-  )
   (wire (pts (xy 69.215 142.875) (xy 69.215 147.955))
     (stroke (width 0) (type default) (color 0 0 0 0))
@@
   )
   (wire (pts (xy 98.425 62.23) (xy 114.935 62.23))
-    (stroke (width 0) (type default) (color 0 0 0 0))
-  )
-  (wire (pts (xy 45.085 104.14) (xy 48.895 104.14))
     (stroke (width 0) (type default) (color 0 0 0 0))
   )
@@
     )
   )
-  (global_label "VBAT2" (shape input) (at 28.575 141.605 90) (fields_autoplaced)
+  (global_label "VBAT1" (shape input) (at 28.575 141.605 90) (fields_autoplaced)
     (effects (font (size 1.27 1.27)) (justify left))
     (property "Intersheet References" "${INTERSHEET_REFS}" (id 0) (at 28.4956 133.5676 90)
@@
     (pin "2")
   )
-  (symbol (lib_id "Device:C_Small") (at 42.545 104.14 270) (unit 1)
-    (in_bom yes) (on_board yes)
-    (property "Reference" "C4" (id 0) (at 41.275 107.315 90)
-      (effects (font (size 1.27 1.27)) (justify left))
-    )
-    (property "Value" "100n" (id 1) (at 41.275 109.22 90)
-      (effects (font (size 1.27 1.27)) (justify left))
-    )
-    (property "Footprint" "Capacitor_SMD:C_0805_2012Metric" (id 2) (at 42.545 104.14 0)
-      (effects (font (size 1.27 1.27)) hide)
-    )
-    (property "Datasheet" "~" (id 3) (at 42.545 104.14 0)
-      (effects (font (size 1.27 1.27)) hide)
-    )
-    (property "Basic/Extended" "Basic" (id 4) (at 42.545 104.14 0)
-      (effects (font (size 1.27 1.27)) hide)
-    )
-    (property "JLCPCB Part #" "C28323" (id 5) (at 42.545 104.14 0)
-      (effects (font (size 1.27 1.27)) hide)
-    )
-    (property "U labosu?" "Da" (id 6) (at 42.545 104.14 0)
-      (effects (font (size 1.27 1.27)) hide)
-    )
-    (pin "1")
-    (pin "2")
-  )
   (symbol (lib_id "Device:R_Small") (at 152.4 94.615 90) (unit 1)
     (in_bom yes) (on_board yes)
@@
     )
     (property "Datasheet" "" (id 3) (at 110.49 147.32 0)
-      (effects (font (size 1.27 1.27)) hide)
-    )
-    (pin "1")
-  )
-  (symbol (lib_id "power:GND") (at 30.48 106.045 0) (unit 1)
-    (in_bom yes) (on_board yes)
-    (property "Reference" "#PWR013" (id 0) (at 30.48 112.395 0)
-      (effects (font (size 1.27 1.27)) hide)
-    )
-    (property "Value" "GND" (id 1) (at 30.607 110.4392 0))
-    (property "Footprint" "" (id 2) (at 30.48 106.045 0)
-      (effects (font (size 1.27 1.27)) hide)
-    )
-    (property "Datasheet" "" (id 3) (at 30.48 106.045 0)
       (effects (font (size 1.27 1.27)) hide)
     )
@@
     (pin "2")
   )
-  (symbol (lib_id "Device:R_Small") (at 34.29 100.33 90) (unit 1)
-    (in_bom yes) (on_board yes)
-    (property "Reference" "R6" (id 0) (at 34.29 98.425 90))
-    (property "Value" "100" (id 1) (at 34.29 100.33 90)
-      (effects (font (size 0.9906 0.9906)))
-    )
-    (property "Footprint" "Resistor_SMD:R_0603_1608Metric" (id 2) (at 34.29 100.33 0)
-      (effects (font (size 1.27 1.27)) hide)
-    )
-    (property "Datasheet" "~" (id 3) (at 34.29 100.33 0)
-      (effects (font (size 1.27 1.27)) hide)
-    )
-    (property "Basic/Extended" "Basic" (id 4) (at 34.29 100.33 0)
-      (effects (font (size 1.27 1.27)) hide)
-    )
-    (property "JLCPCB Part #" "C17414" (id 5) (at 34.29 100.33 0)
-      (effects (font (size 1.27 1.27)) hide)
-    )
-    (property "U labosu?" "Da" (id 6) (at 34.29 100.33 0)
-      (effects (font (size 1.27 1.27)) hide)
-    )
-    (pin "1")
-    (pin "2")
-  )
   (symbol (lib_id "power:GND") (at 110.49 158.75 0) (unit 1)
     (in_bom yes) (on_board yes) (fields_autoplaced)
@@
     )
     (pin "1")
-  )
-  (symbol (lib_id "Switch:SW_Push") (at 42.545 100.33 0) (unit 1)
-    (in_bom yes) (on_board yes)
-    (property "Reference" "SW3" (id 0) (at 42.545 95.25 0))
-    (property "Value" "SW_Push" (id 1) (at 42.545 95.4024 0)
-      (effects (font (size 1.27 1.27)) hide)
-    )
-    (property "Footprint" "Button_Switch_SMD:SW_SPST_TL3342" (id 2) (at 42.545 95.25 0)
-      (effects (font (size 1.27 1.27)) hide)
-    )
-    (property "Datasheet" "~" (id 3) (at 42.545 95.25 0)
-      (effects (font (size 1.27 1.27)) hide)
-    )
-    (property "Basic/Extended" "Basic" (id 4) (at 42.545 100.33 0)
-      (effects (font (size 1.27 1.27)) hide)
-    )
-    (property "JLCPCB Part #" "C307331" (id 5) (at 42.545 100.33 0)
-      (effects (font (size 1.27 1.27)) hide)
-    )
-    (property "U labosu?" "Ne" (id 6) (at 42.545 100.33 0)
-      (effects (font (size 1.27 1.27)) hide)
-    )
-    (pin "1")
-    (pin "2")
   )
   (symbol (lib_id "power:PWR_FLAG") (at 26.67 123.19 0) (unit 1)
@@
       (reference "#PWR012") (unit 1) (value "GND") (footprint "")
     )
-    (path "/29a86eae-b86b-4d15-b4ef-23047eb09446"
-      (reference "#PWR013") (unit 1) (value "GND") (footprint "")
-    )
     (path "/96de6c56-95bd-4bef-b242-a01019dc90f5"
       (reference "#PWR014") (unit 1) (value "GND") (footprint "")
@@
       (reference "C3") (unit 1) (value "100n") (footprint "Capacitor_SMD:C_0805_2012Metric")
     )
-    (path "/054adfe7-200d-4f98-a8b0-7f9f5e050ecd"
-      (reference "C4") (unit 1) (value "100n") (footprint "Capacitor_SMD:C_0805_2012Metric")
-    )
     (path "/4bdbd67c-fc66-41a9-aa66-e5f5f4127563"
       (reference "C5") (unit 1) (value "22u / 16V") (footprint "Capacitor_SMD:C_1210_3225Metric")
@@
       (reference "R5") (unit 1) (value "220") (footprint "Resistor_SMD:R_0603_1608Metric")
     )
-    (path "/7b7e5c9e-a29f-4968-b447-f6d172770aa4"
-      (reference "R6") (unit 1) (value "100") (footprint "Resistor_SMD:R_0603_1608Metric")
-    )
     (path "/d03e3188-cc2d-4da7-b438-ae7e092bd132"
       (reference "R7") (unit 1) (value "100") (footprint "Resistor_SMD:R_0603_1608Metric")
@@
       (reference "SW2") (unit 1) (value "SW_Push") (footprint "Footprint:Omron_B3F-12x12mm")
     )
-    (path "/a11bfb73-f8ea-4766-8e87-c59e9f3162b4"
-      (reference "SW3") (unit 1) (value "SW_Push") (footprint "Button_Switch_SMD:SW_SPST_TL3342")
-    )
     (path "/665f548c-e32f-4b45-a237-85cb92f121a3"

Commit message: update
Parts:
- removed J2: ST7789, Footprint:ST7789, symbol Connector_Generic:Conn_01x07
- removed R1, R2, R3, R5: 220, Resistor_SMD:R_0603_1608Metric, symbol Device:R_Small
- added J2: OLED, Footprint:OLED, symbol Connector_Generic:Conn_01x04
- C1, C2, C3, CD1, CD2: footprint Capacitor_SMD:C_0805_2012Metric -> Capacitor_SMD:C_0603_1608Metric
Connections:
- net +3V3: now also J2.2 (Pin_2)
- net +5V: no longer C3.1, U1.20 (AREF)
- net GND: now also J3.1 (Pin_1), J2.1 (Pin_1); no longer J3.3 (Pin_3)
- net MOSFET2: now also U1.14 (PB2); no longer U1.9 (PD5)
- net MOSFET3: now also U1.11 (PD7); no longer U1.10 (PD6)
- net MOSFET4: now also U1.10 (PD6); no longer U1.11 (PD7)
- net TX: now also J3.3 (Pin_3); no longer J3.1 (Pin_1)
- net BUZZER: now reaches LS1.1
- net BUZZER: now also U1.9 (PD5); no longer U1.14 (PB2)
- net IBAT1 renamed SDA
- net SDA: now also J2.4 (Pin_4)
- net IBAT2 renamed SCL
- net SCL: now also J2.3 (Pin_3)
- net IBAT3: no longer names the net of U1.19 (ADC6)
- net IBAT4: no longer names the net of U1.22 (ADC7)
- net INT0 renamed PD2/INT0
- net INT1 renamed PD3/INT1
- net MOSI renamed PB3
- net PB0: no longer names the net of U1.12 (PB0)
- net PB1: no longer names the net of U1.13 (PB1)
- new net AREF: C3.1, U1.20 (AREF)
- no-connect marks 1 -> 4
Other:
- note added: "D2"
- note added: "D3"
- note added: "MISO"
- note added: "MOSI"
- note added: "RESET"
- note added: "SCK"
- note removed: "ST7789"
- moved on the sheet: C1, C2, C3, J1, J3, L1, LS1, R4, U1, Y1

Commit message: update
Parts:
- H1, H2, H3, H4: symbol Mechanical:MountingHole -> Mechanical:MountingHole_Pad
Connections:
- net RX: now also J3.3 (Pin_3), U1.30 (PD0); no longer J3.2 (Pin_2), U1.31 (PD1)
- net TX: now also J3.2 (Pin_2), U1.31 (PD1); no longer J3.3 (Pin_3), U1.30 (PD0)
- no-connect marks 4 -> 8
Other:
- moved on the sheet: C1, C2, C3, J1, J2, J3, L1, LS1, R4, U1, Y1

Commit message: update
Other:
- note added: "- logo - qrcode - email - ime i verzija"
Changed lines of the file:
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@@
     (effects (font (size 1.27 1.27)) (justify left bottom))
+  )
+  (text "- logo\n- qrcode\n- email\n- ime i verzija" (at 24.13 189.23 0)
+    (effects (font (size 2 2)) (justify left bottom))
   )
   (text "D3" (at 208.28 139.7 0)
