File: KiCAD_Files/BatteryDischargerV1.kicad_sch (KiCad schematic)
At the start: 31 parts, among them J1 USBasp, J2 OLED, J3 UART, SW1 SW_Push, SW2 SW_Push, U1 ATmega328-A, U2 AMS1117-3.3, U3 MT3608, Y1 16MHz

Commit message: update
Other:
- note added: "- dodati 100k pull-down otpornike na sve analogne ulaze - logo - qrcode - email - ime i verzija"
- note removed: "- logo - qrcode - email - ime i verzija"
Changed lines of the file:
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@@
     (effects (font (size 1.27 1.27)) (justify left bottom))
   )
-  (text "- logo\n- qrcode\n- email\n- ime i verzija" (at 24.13 189.23 0)
+  (text "- dodati 100k pull-down otpornike na sve analogne ulaze\n- logo\n- qrcode\n- email\n- ime i verzija"
+    (at 17.78 193.675 0)
     (effects (font (size 2 2)) (justify left bottom))
   )

Commit message: kicad7
Other:
- note added: "- dodati 100k pull-down otpornike na sve analogne ulaze - reverse polarity dioda / mosfet kod svake baterije za reverse polarity protection - logo - qrcode - email - ime i verzija"
- note removed: "- dodati 100k pull-down otpornike na sve analogne ulaze - logo - qrcode - email - ime i verzija"
